File: PCB/Bird3Controller/Bird3Controller.kicad_sch (KiCad schematic)
At the start: 49 parts, among them IC2 LM3519MK-20_NOPB, IC3 LM3405AXMY_NOPB, J1 Bird 3 24-pin Connector, J2 TXW154028S0 Connector, J3 2171800001, SW1 SW_Boot, SW2 SW_Reset, U1 ESP32-S3-WROOM-1, U3 SN65HVD231, U4 LMR36520ADDAR

Commit message: Final Rev1 schematic update
Parts:
- R13: Manufacturer_Part_Number CRCW0805150KFKEAC -> CRCW080543K2FKEAC; Mouser Part Number 71-CRCW0805150KFKEAC -> 71-CRCW080543K2FKEAC
