File: PCB/Bird3Controller_Rev2/Bird3Controller.kicad_sch (KiCad schematic)
At the start: 52 parts, among them IC1 M24C08-RMN6TP, J1 Bird 3 24-pin Connector, J2 TXW154028S0 Connector, J3 87832-2220, Q1 2N7002A, SW1 SW_Boot, SW2 SW_Reset, U1 ESP32-S3-WROOM-1, U3 SN65HVD231, U4 LMR36520ADDAR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

Commit message: Fix part number that referred to 0.402ohm resistor instead of the correct 0.200ohm value
Parts:
- R7: Digikey Part Number 1712-RLC73K2AR402FTDCT-ND -> (none); Manufacturer_Part_Number RLC73K2AR402FTDF -> RLC73K2AR20FTDF; Mouser Part Number 279-RLC73K2AR402FTDF -> 279-RLC73K2AR20FTDF; Mouser Price/Stock https://www.mouser.com/ProductDetail/TE-Connectivity-CGS/RLC73K2AR402FTDF?qs=9vOqFld9vZX6KRPnzoA4cw%3D%3D -> https://www.mouser.com/ProductDetail/TE-Connectivity-CGS/RLC73K2AR20FTDF?qs=9vOqFld9vZWQ3oqbYNtegw%3D%3D
Changed lines of the file:
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@@
 			)
 		)
-		(property "Mouser Part Number" "279-RLC73K2AR402FTDF"
+		(property "Mouser Part Number" "279-RLC73K2AR20FTDF"
 			(at 165.1 158.75 0)
 			(effects
@@
 			)
 		)
-		(property "Manufacturer_Part_Number" "RLC73K2AR402FTDF"
+		(property "Manufacturer_Part_Number" "RLC73K2AR20FTDF"
 			(at 167.64 172.72 0)
 			(effects
@@
 			)
 		)
-		(property "Digikey Part Number" "1712-RLC73K2AR402FTDCT-ND"
+		(property "Digikey Part Number" ""
 			(at 167.64 175.26 0)
 			(effects
@@
 			)
 		)
-		(property "Mouser Price/Stock" "https://www.mouser.com/ProductDetail/TE-Connectivity-CGS/RLC73K2AR402FTDF?qs=9vOqFld9vZX6KRPnzoA4cw%3D%3D"
+		(property "Mouser Price/Stock" "https://www.mouser.com/ProductDetail/TE-Connectivity-CGS/RLC73K2AR20FTDF?qs=9vOqFld9vZWQ3oqbYNtegw%3D%3D"
 			(at 165.1 158.75 0)
 			(effects
