File: PCB/Bird3Controller_Rev3/Bird3Controller.kicad_pcb (KiCad board)
At the start: 2 copper layers, 43 x 108 mm, 61 parts, among them IC1 M24C08-RMN6TP, IC2 AP63203WU-7, J1 Bird 3 24-pin Connector, J2 TXW154028S0 Connector, J3 87832-2220, Q1 2N7002A, SW1 SW_Boot, SW2 SW_Reset, U1 ESP32-S3-WROOM-1, U3 SN65HVD231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

Commit message: Optimize ground plane/vias
Parts:
- J4: value ~ -> Adafruit USB-C Breakout
Routing:
- net +3V3: track 215.8 -> 212.7 mm
- net GND: track 382.2 -> 379.3 mm, vias 114 -> 145
- net /CAN_TX: track 39.2 -> 38.4 mm
- net /BR1: track 72.0 -> 72.6 mm
- net /CAN_RX: track 36.8 -> 36.3 mm
